File: forZero_schematy/cluster_plugs.kicad_sch (KiCad schematic)
At the start: 6 parts, among them J2 43045-0800, J3 43045-0621, J4 43045-0400, J5 Barrel_Jack_Switch

Commit message: Wprowadzenie poprawek PCB
Connections:
- net CLUSTER_SENSOR: now also J2.4; no longer J2.8
- net CLUSTER_BREAK_PADS renamed CLUSTER_BRAKE_PADS
- new net CLUSTER_TCR: J2.8
- no-connect marks 4 -> 3
Changed lines of the file:
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@@
-	)
-	(no_connect
-		(at 170.18 111.76)
 	)
 	(no_connect
@@
 	(wire
 		(pts
-			(xy 193.04 111.76) (xy 190.5 111.76)
-		)
-		(stroke
-			(width 0)
-			(type default)
-		)
-	)
-	(wire
-		(pts
 			(xy 85.09 77.47) (xy 86.36 77.47)
 		)
@@
 	(wire
 		(pts
+			(xy 167.64 111.76) (xy 170.18 111.76)
+		)
+		(stroke
+			(width 0)
+			(type default)
+		)
+	)
+	(wire
+		(pts
 			(xy 167.64 114.3) (xy 170.18 114.3)
 		)
@@
 	(wire
 		(pts
+			(xy 190.5 111.76) (xy 193.04 111.76)
+		)
+		(stroke
+			(width 0)
+			(type default)
+		)
+	)
+	(wire
+		(pts
 			(xy 101.6 111.76) (xy 99.06 111.76)
 		)
@@
 		)
 	)
+	(global_label "CLUSTER_TCR"
+		(shape input)
+		(at 193.04 111.76 0)
+		(fields_autoplaced yes)
+		(effects
+			(font
+				(size 1.27 1.27)
+			)
+			(justify left)
+		)
+		(property "Intersheetrefs" "${INTERSHEET_REFS}"
+			(at 208.7251 111.76 0)
+			(effects
+				(font
+					(size 1.27 1.27)
+				)
+				(justify left)
+				(hide yes)
+			)
+		)
+	)
 	(global_label "CLUSTER_ABS"
 		(shape input)
@@
 	(global_label "CLUSTER_SENSOR"
 		(shape input)
-		(at 193.04 111.76 0)
-		(fields_autoplaced yes)
-		(effects
-			(font
-				(size 1.27 1.27)
-			)
-			(justify left)
-		)
-		(property "Intersheetrefs" "${INTERSHEET_REFS}"
-			(at 212.7165 111.76 0)
-			(effects
-				(font
-					(size 1.27 1.27)
-				)
-				(justify left)
-				(hide yes)
-			)
-		)
-	)
-	(global_label "CLUSTER_BREAK_PADS"
+		(at 167.64 111.76 180)
+		(fields_autoplaced yes)
+		(effects
+			(font
+				(size 1.27 1.27)
+			)
+			(justify right)
+		)
+		(property "Intersheetrefs" "${INTERSHEET_REFS}"
+			(at 147.9635 111.76 0)
+			(effects
+				(font
+					(size 1.27 1.27)
+				)
+				(justify right)
+				(hide yes)
+			)
+		)
+	)
+	(global_label "CLUSTER_BRAKE_PADS"
 		(shape input)
 		(at 193.04 114.3 0)
