File: forZero_schematy/usb_and_can_controler.kicad_sch (KiCad schematic)
At the start: 15 parts, among them IC4 AP7347DQ-33W5-7, IC5 MCP2562-E_SN, J1 USB_C_Receptacle_USB2.0_16P

Commit message: Wprowadzenie poprawek PCB
Connections:
- net 5V_USB: no longer names the net of F1.2, J1.A4 (VBUS), J1.A9 (VBUS), J1.B4 (VBUS), J1.B9 (VBUS)
Changed lines of the file:
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@@
-	)
-	(junction
-		(at 60.96 63.5)
-		(diameter 0)
-		(color 0 0 0 0)
 	)
 	(junction
@@
 	(junction
 		(at 181.61 67.31)
+		(diameter 0)
+		(color 0 0 0 0)
+	)
+	(junction
+		(at 60.96 53.34)
 		(diameter 0)
 		(color 0 0 0 0)
@@
 	(wire
 		(pts
-			(xy 60.96 52.07) (xy 60.96 54.61)
-		)
-		(stroke
-			(width 0)
-			(type default)
-		)
-	)
-	(wire
-		(pts
 			(xy 232.41 67.31) (xy 236.22 67.31)
 		)
@@
 	(wire
 		(pts
-			(xy 60.96 63.5) (xy 63.5 63.5)
-		)
-		(stroke
-			(width 0)
-			(type default)
-		)
-	)
-	(wire
-		(pts
 			(xy 236.22 62.23) (xy 241.3 62.23)
 		)
@@
 	(wire
 		(pts
+			(xy 63.5 50.8) (xy 60.96 50.8)
+		)
+		(stroke
+			(width 0)
+			(type default)
+		)
+	)
+	(wire
+		(pts
 			(xy 115.57 115.57) (xy 118.11 115.57)
 		)
@@
 	(wire
 		(pts
+			(xy 60.96 53.34) (xy 60.96 54.61)
+		)
+		(stroke
+			(width 0)
+			(type default)
+		)
+	)
+	(wire
+		(pts
 			(xy 39.37 102.87) (xy 39.37 104.14)
 		)
@@
 	(wire
 		(pts
+			(xy 60.96 53.34) (xy 63.5 53.34)
+		)
+		(stroke
+			(width 0)
+			(type default)
+		)
+	)
+	(wire
+		(pts
 			(xy 123.19 86.36) (xy 127 86.36)
 		)
@@
 		(pts
 			(xy 60.96 62.23) (xy 60.96 63.5)
+		)
+		(stroke
+			(width 0)
+			(type default)
+		)
+	)
+	(wire
+		(pts
+			(xy 60.96 50.8) (xy 60.96 53.34)
 		)
 		(stroke
@@
 	(global_label "5V"
 		(shape output)
-		(at 60.96 52.07 90)
+		(at 63.5 50.8 0)
 		(fields_autoplaced yes)
 		(effects
@@
 		)
 		(property "Intersheetrefs" "${INTERSHEET_REFS}"
-			(at 60.96 46.7867 90)
+			(at 68.7833 50.8 0)
 			(effects
 				(font
@@
 	(global_label "5V_USB"
 		(shape output)
-		(at 63.5 63.5 0)
+		(at 63.5 53.34 0)
 		(fields_autoplaced yes)
 		(effects
@@
 		)
 		(property "Intersheetrefs" "${INTERSHEET_REFS}"
-			(at 73.5609 63.5 0)
+			(at 73.5609 53.34 0)
 			(effects
 				(font
