File: forZero_schematy/forZero.kicad_sch (KiCad schematic)
At the start: 24 parts, among them IC3 STM32F105RBT6, Y1 25MHz

Commit message: Wprowadzenie poprawek PCB
Connections:
- net BREAK_PADS is gone; now on net ABS: IC3.26 (PB0)
- net ABS: no longer IC3.27 (PB1)
- net SENSOR: now also IC3.29 (PB10); no longer IC3.22 (PA6)
- net TCR: now reaches IC3.24 (PC4)
- net BRAKE_PADS: now reaches IC3.25 (PC5)
- no-connect marks 29 -> 28
Other:
- note added: "5mA each LEDs"
- moved on the sheet: R41
Changed lines of the file:
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@@
 		)
 	)
+	(text "5mA each LEDs "
+		(exclude_from_sim no)
+		(at 235.204 81.026 0)
+		(effects
+			(font
+				(size 1.27 1.27)
+			)
+		)
+	)
 	(text "Stm32 configuration"
 		(exclude_from_sim no)
@@
 	)
 	(no_connect
-		(at 132.08 54.61)
+		(at 127 128.27)
 	)
 	(no_connect
-		(at 132.08 128.27)
+		(at 132.08 54.61)
 	)
 	(no_connect
-		(at 144.78 128.27)
+		(at 124.46 128.27)
 	)
 	(no_connect
@@
 	)
 	(no_connect
-		(at 134.62 128.27)
-	)
-	(no_connect
 		(at 106.68 105.41)
 	)
 	(no_connect
-		(at 124.46 128.27)
-	)
-	(no_connect
 		(at 137.16 54.61)
 	)
@@
 	)
 	(no_connect
+		(at 139.7 128.27)
+	)
+	(no_connect
 		(at 106.68 74.93)
 	)
@@
 	(wire
 		(pts
-			(xy 246.38 96.52) (xy 246.38 100.33)
-		)
-		(stroke
-			(width 0)
-			(type default)
-		)
-	)
-	(wire
-		(pts
-			(xy 44.45 133.35) (xy 44.45 129.54)
+			(xy 144.78 128.27) (xy 144.78 130.81)
 		)
 		(stroke
@@
 	(wire
 		(pts
-			(xy 114.3 53.34) (xy 114.3 54.61)
+			(xy 137.16 128.27) (xy 137.16 130.81)
 		)
 		(stroke
@@
 	(wire
 		(pts
-			(xy 163.83 71.12) (xy 166.37 71.12)
+			(xy 246.38 96.52) (xy 246.38 100.33)
 		)
 		(stroke
@@
 	(wire
 		(pts
-			(xy 264.16 96.52) (xy 264.16 100.33)
+			(xy 44.45 133.35) (xy 44.45 129.54)
 		)
 		(stroke
@@
 	(wire
 		(pts
-			(xy 34.29 120.65) (xy 34.29 124.46)
+			(xy 114.3 53.34) (xy 114.3 54.61)
 		)
 		(stroke
@@
 	(wire
 		(pts
-			(xy 71.12 121.92) (xy 71.12 123.19)
+			(xy 163.83 71.12) (xy 166.37 71.12)
 		)
 		(stroke
@@
 	(wire
 		(pts
-			(xy 129.54 52.07) (xy 129.54 54.61)
+			(xy 264.16 96.52) (xy 264.16 100.33)
 		)
 		(stroke
@@
 	(wire
 		(pts
-			(xy 152.4 52.07) (xy 152.4 54.61)
+			(xy 34.29 120.65) (xy 34.29 124.46)
 		)
 		(stroke
@@
 	(wire
 		(pts
-			(xy 102.87 72.39) (xy 106.68 72.39)
+			(xy 71.12 121.92) (xy 71.12 123.19)
 		)
 		(stroke
@@
 	(wire
 		(pts
-			(xy 34.29 69.85) (xy 34.29 71.12)
+			(xy 129.54 52.07) (xy 129.54 54.61)
 		)
 		(stroke
@@
 	(wire
 		(pts
-			(xy 149.86 128.27) (xy 149.86 129.54)
+			(xy 152.4 52.07) (xy 152.4 54.61)
 		)
 		(stroke
@@
 	(wire
 		(pts
-			(xy 124.46 52.07) (xy 124.46 54.61)
+			(xy 102.87 72.39) (xy 106.68 72.39)
 		)
 		(stroke
@@
 	(wire
 		(pts
-			(xy 129.54 130.81) (xy 129.54 128.27)
+			(xy 34.29 69.85) (xy 34.29 71.12)
 		)
 		(stroke
@@
 	(wire
 		(pts
-			(xy 34.29 125.73) (xy 34.29 124.46)
+			(xy 149.86 128.27) (xy 149.86 129.54)
 		)
 		(stroke
@@
 	(wire
 		(pts
-			(xy 92.71 102.87) (xy 95.25 102.87)
+			(xy 124.46 52.07) (xy 124.46 54.61)
 		)
 		(stroke
@@
 	(wire
 		(pts
-			(xy 137.16 130.81) (xy 137.16 128.27)
+			(xy 34.29 125.73) (xy 34.29 124.46)
 		)
 		(stroke
@@
 	(wire
 		(pts
-			(xy 127 130.81) (xy 127 128.27)
+			(xy 92.71 102.87) (xy 95.25 102.87)
 		)
 		(stroke
@@
 	(wire
 		(pts
-			(xy 142.24 128.27) (xy 142.24 135.89)
+			(xy 142.24 128.27) (xy 142.24 139.7)
 		)
 		(stroke
@@
 	(wire
 		(pts
-			(xy 139.7 130.81) (xy 139.7 128.27)
-		)
-		(stroke
-			(width 0)
-			(type default)
-		)
-	)
-	(wire
-		(pts
 			(xy 34.29 71.12) (xy 39.37 71.12)
 		)
@@
 	(wire
 		(pts
+			(xy 132.08 128.27) (xy 132.08 130.81)
+		)
+		(stroke
+			(width 0)
+			(type default)
+		)
+	)
+	(wire
+		(pts
 			(xy 69.85 66.04) (xy 69.85 68.58)
 		)
@@
 	(wire
 		(pts
+			(xy 134.62 128.27) (xy 134.62 130.81)
+		)
+		(stroke
+			(width 0)
+			(type default)
+		)
+	)
+	(wire
+		(pts
 			(xy 119.38 128.27) (xy 119.38 138.43)
 		)
@@
 		)
 	)
+	(wire
+		(pts
+			(xy 129.54 128.27) (xy 129.54 130.81)
+		)
+		(stroke
+			(width 0)
+			(type default)
+		)
+	)
 	(global_label "COOL_LVL"
 		(shape output)
@@
 	(global_label "ABS"
 		(shape output)
-		(at 139.7 130.81 270)
+		(at 137.16 130.81 270)
 		(fields_autoplaced yes)
 		(effects
@@
 		)
 		(property "Intersheetrefs" "${INTERSHEET_REFS}"
-			(at 139.7 137.3633 90)
+			(at 137.16 137.3633 90)
 			(effects
 				(font
@@
 		)
 	)
+	(global_label "TCR"
+		(shape output)
+		(at 132.08 130.81 270)
+		(fields_autoplaced yes)
+		(effects
+			(font
+				(size 1.27 1.27)
+			)
+			(justify right)
+		)
+		(property "Intersheetrefs" "${INTERSHEET_REFS}"
+			(at 132.08 137.3028 90)
+			(effects
+				(font
+					(size 1.27 1.27)
+				)
+				(justify right)
+				(hide yes)
+			)
+		)
+	)
 	(global_label "SENSOR"
 		(shape output)
-		(at 127 130.81 270)
+		(at 144.78 130.81 270)
 		(fields_autoplaced yes)
 		(effects
@@
 		)
 		(property "Intersheetrefs" "${INTERSHEET_REFS}"
-			(at 127 141.2942 90)
+			(at 144.78 141.2942 90)
 			(effects
 				(font
@@
 		)
 	)
-	(global_label "BREAK_PADS"
+	(global_label "BRAKE_PADS"
 		(shape output)
-		(at 137.16 130.81 270)
+		(at 134.62 130.81 270)
 		(fields_autoplaced yes)
 		(effects
@@
 		)
 		(property "Intersheetrefs" "${INTERSHEET_REFS}"
-			(at 137.16 145.6485 90)
+			(at 134.62 145.6485 90)
 			(effects
 				(font
@@
 	(symbol
 		(lib_id "Device:R")
-		(at 142.24 139.7 0)
+		(at 142.24 143.51 0)
 		(unit 1)
 		(exclude_from_sim no)
@@
 		(fields_autoplaced yes)
 		(property "Reference" "R41"
-			(at 144.78 138.4299 0)
+			(at 144.78 142.2399 0)
 			(effects
 				(font
@@
 		)
 		(property "Value" "9.1k"
-			(at 144.78 140.9699 0)
+			(at 144.78 144.7799 0)
 			(effects
 				(font
@@
 		)
 		(property "Footprint" "Resistor_SMD:R_0805_2012Metric_Pad1.20x1.40mm_HandSolder"
-			(at 140.462 139.7 90)
+			(at 140.462 143.51 90)
 			(effects
 				(font
@@
 		)
 		(property "Datasheet" "~"
-			(at 142.24 139.7 0)
+			(at 142.24 143.51 0)
 			(effects
 				(font
@@
 		)
 		(property "Description" "Resistor"
-			(at 142.24 139.7 0)
+			(at 142.24 143.51 0)
 			(effects
 				(font
@@
 	(symbol
 		(lib_id "power:GND")
-		(at 142.24 143.51 0)
+		(at 142.24 147.32 0)
 		(unit 1)
 		(exclude_from_sim no)
@@
 		(dnp no)
 		(property "Reference" "#PWR057"
-			(at 142.24 149.86 0)
+			(at 142.24 153.67 0)
 			(effects
 				(font
@@
 		)
 		(property "Value" "GND"
-			(at 142.494 148.336 90)
+			(at 142.24 151.13 0)
 			(effects
 				(font
@@
 		)
 		(property "Footprint" ""
-			(at 142.24 143.51 0)
+			(at 142.24 147.32 0)
 			(effects
 				(font
@@
 		)
 		(property "Datasheet" ""
-			(at 142.24 143.51 0)
+			(at 142.24 147.32 0)
 			(effects
 				(font
@@
 		)
 		(property "Description" "Power symbol creates a global label with name \"GND\" , ground"
-			(at 142.24 143.51 0)
+			(at 142.24 147.32 0)
 			(effects
 				(font

Commit message: Wykonano finalne PCB dla forZero_1v0
Parts:
- renumbered ERR1 to ERROR1
Changed lines of the file:
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@@
 		(on_board yes)
 		(dnp no)
-		(property "Reference" "ERR1"
+		(property "Reference" "ERROR1"
 			(at 267.97 102.87 90)
 			(effects
@@
 			(project "forZero"
 				(path "/be6e4903-743e-4026-a4b6-03f90da5b2a5"
-					(reference "ERR1")
+					(reference "ERROR1")
 					(unit 1)
 				)
